Commit message: set lidar

File: src/articubot_one/description/lidar.xacro (robot description, xacro)
@@ -4,10 +4,10 @@
         <parent link="chassis"/>
         <child link="laser_frame"/>
-        <origin xyz="0 0 0.115" rpy="0 0 0"/>
+        <origin xyz="0 0 0.195" rpy="0 0 0"/>
     </joint>
     <link name="laser_frame">
         <visual>
             <geometry>
-                <cylinder radius="0.05" length="0.01"/>
+                <cylinder radius="0.05" length="0.07"/>
             </geometry>
             <material name="black"/>
@@ -15,5 +15,5 @@
         <collision>
             <geometry>
-                <cylinder radius="0.05" length="0.01"/>
+                <cylinder radius="0.05" length="0.07"/>
             </geometry>
         </collision>

File: src/articubot_one/description/robot.urdf.xacro (robot description, xacro)
@@ -5,4 +5,4 @@
     <xacro:include filename="gazebo_control.xacro" />
     <xacro:include filename="lidar.xacro" />
-    <xacro:include filename="gripper.xacro" />
+    <!-- <xacro:include filename="gripper.xacro" /> -->
 </robot>
