Commit message: can navigation already launch pass turtle

File: src/articubot_one/description/gripper.xacro (robot description, xacro)
@@ -4,5 +4,5 @@
     <link name="gripper_base">
         <visual>
-            <origin xyz="0 0 0" rpy="0 0 0"/>
+            <origin xyz="1 1.3 0.35" rpy="0 0 0"/>
             <geometry>
                 <box size="0.35 0.05 0.05"/>
@@ -24,5 +24,5 @@
     <link name="gripper_finger_left">
         <visual>
-            <origin xyz="-0.075 0 0" rpy="0 0 0"/>
+            <origin xyz="-0.095 1 0" rpy="0 0 0"/>
             <geometry>
                 <box size="0.02 0.1 0.02"/>
@@ -44,5 +44,5 @@
     <link name="gripper_finger_right">
         <visual>
-            <origin xyz="0.075 0 0" rpy="0 0 0"/>
+            <origin xyz="0.095 1 0" rpy="0 0 0"/>
             <geometry>
                 <box size="0.02 0.1 0.02"/>
@@ -65,5 +65,5 @@
         <parent link="chassis"/>
         <child link="gripper_base"/>
-        <origin xyz="0.25 0 0.05" rpy="0 0 1.57"/>
+        <origin xyz="0 0 0.14" rpy="0 0 1.57"/>
         <axis xyz="0 0 1"/>
         <limit effort="10" lower="0" upper="0.13" velocity="0.1"/>
