Commit message: keyboard but cant use gripper

File: src/articubot_one/description/gazebo_control.xacro (robot description, xacro)
@@ -1,4 +1,11 @@
 <?xml version="1.0"?>
 <robot xmlns:xacro="http://www.ros.org/wiki/xacro">
+    <xacro:macro name="robot_controller">
+        <gazebo>
+            <plugin name="gazebo_ros2_control_robot" filename="libgazebo_ros2_control.so">
+                <parameters>$(find articubot_one)/config/controller.yaml</parameters>
+            </plugin>
+        </gazebo>
+    </xacro:macro>
     <gazebo>
         <plugin name='back_wheel' filename='libgazebo_ros_diff_drive.so'>
@@ -35,3 +42,21 @@
         </plugin>
     </gazebo>
+    <gazebo>
+        <plugin name="gazebo_ros_joint_state_publisher" filename="libgazebo_ros_joint_state_publisher.so">
+            <update_rate>20</update_rate>
+            <joint_name>gripper_finger_left_joint</joint_name>
+            <joint_name>gripper_vertical_joint</joint_name>
+            <joint_name>gripper_finger_right_joint</joint_name>
+        </plugin>
+        <plugin name="gazebo_ros_joint_pose_trajectory" filename="libgazebo_ros_joint_pose_trajectory.so">
+            <update_rate>20</update_rate>
+        </plugin>
+	<!-- Load transmission plugin -->
+    	<plugin name="transmission" filename="libgazebo_ros2_control.so">
+      	    <robotNamespace>/</robotNamespace>
+      	    <controlPeriod>0.001</controlPeriod>
+            <robotParam>articubot_one</robotParam>
+            <robotSimType>gazebo_ros_control/DefaultRobotHWSim</robotSimType>
+    	</plugin>
+    </gazebo>
 </robot>

File: src/articubot_one/description/gripper.xacro (robot description, xacro)
@@ -4,9 +4,9 @@
     <link name="gripper_base">
         <visual>
-            <origin xyz="1 1.3 0.35" rpy="0 0 0"/>
+            <origin xyz="0 0.23 -0.05" rpy="0 0 0"/>
             <geometry>
-                <box size="0.35 0.05 0.05"/>
+                <box size="0.45 0.05 0.03"/>
             </geometry>
-            <material name="gray"/>
+            <material name="blue"/>
         </visual>
         <collision>
@@ -24,13 +24,13 @@
     <link name="gripper_finger_left">
         <visual>
-            <origin xyz="-0.095 1 0" rpy="0 0 0"/>
+            <origin xyz="-0.095 0.38 -0.05" rpy="0 0 0"/>
             <geometry>
-                <box size="0.02 0.1 0.02"/>
+                <box size="0.025 0.12 0.035"/>
             </geometry>
-            <material name="orange"/>
+            <material name="blue"/>
         </visual>
         <collision>
             <geometry>
-                <box size="0.02 0.1 0.02"/>
+                <box size="0.025 0.12 0.025"/>
             </geometry>
         </collision>
@@ -44,13 +44,13 @@
     <link name="gripper_finger_right">
         <visual>
-            <origin xyz="0.095 1 0" rpy="0 0 0"/>
+            <origin xyz="0.095 0.38 -0.05" rpy="0 0 0"/>
             <geometry>
-                <box size="0.02 0.1 0.02"/>
+                <box size="0.025 0.12 0.025"/>
             </geometry>
-            <material name="orange"/>
+            <material name="blue"/>
         </visual>
         <collision>
             <geometry>
-                <box size="0.02 0.1 0.02"/>
+                <box size="0.025 0.12 0.025"/>
             </geometry>
         </collision>
@@ -89,13 +89,13 @@
     <!-- Gazebo Simulation for Gripper -->
     <gazebo reference="gripper_base">
-        <material>Gazebo/Gray</material>
+        <material>Gazebo/Blue</material>
         <gravity>true</gravity>
     </gazebo>
     <gazebo reference="gripper_finger_left">
-        <material>Gazebo/Orange</material>
+        <material>Gazebo/Blue</material>
         <gravity>true</gravity>
     </gazebo>
     <gazebo reference="gripper_finger_right">
-        <material>Gazebo/Orange</material>
+        <material>Gazebo/Blue</material>
         <gravity>true</gravity>
     </gazebo>

File: src/articubot_one/description/robot.urdf.xacro (robot description, xacro)
@@ -3,6 +3,20 @@
     <xacro:include filename="inertial_macros.xacro" />
     <xacro:include filename="robot_car.xacro" />
-    <xacro:include filename="gazebo_control.xacro" />
+    <xacro:include filename="gazebo_control.xacro" />,
     <xacro:include filename="lidar.xacro" />
+    <xacro:include filename="gripper.xacro" />
+    <!-- <xacro:include filename="gripperja.xacro" /> -->
+    <!-- <xacro:include filename="arm_tr.xacro" /> -->
+    <!-- <xacro:include filename="gripper_tr.xacro" />  -->
     <!-- <xacro:include filename="gripper.xacro" /> -->
+     <!-- <xacro:include filename="testgripper.xacro" /> -->
+    <!-- <ros2_control name="gripper_robot_gazebo_system" type="system">
+        <hardware>
+            <plugin>gazebo_ros2_control/GazeboSystem</plugin>
+        </hardware>
+        <xacro:arm_tr/>
+        <xacro:gripper1_tr/>
+        <xacro:gripper2_tr/>
+    </ros2_control>
+    <xacro:robot_controller/> -->
 </robot>
